File: kicad_control/busmodule.kicad_sch (KiCad schematic)
At the start: 8 parts, among them U11 74LS374, U12 74LS163, U13 74LS163, U14 74LS163, U15 74LS163, U16 74LS244, U17 74LS244, U18 74LS374

Commit message: Redoing control board because of pipeline blunder. This also is the last version with the distinct program counter.
Parts:
- renumbered U12 to U1, U13 to U2, U14 to U3, U15 to U4, U16 to U5, U17 to U6, U11 to U7, U18 to U8
Connections:
- net +5V: now also U1.10 (CET), U1.7 (CEP), U2.10 (CET), U2.7 (CEP), U3.10 (CET), U3.7 (CEP), U4.10 (CET), U4.7 (CEP)
- net AD12: no longer U3.15 (TC), U4.2 (CP), U4.4 (D1), U4.5 (D2), U4.6 (D3), U8.14 (D5), U8.17 (D6), U8.18 (D7)
- net GND: now also U5.19 (OEb), U6.19 (OEb)
- net ~{pctoaddr}: no longer U5.19 (OEb), U6.19 (OEb)
- new net: U3.15 (TC), U4.2 (CP)
- new net AD13: U4.4 (D1), U8.14 (D5)
- new net AD14: U4.5 (D2), U8.17 (D6)
- new net AD15: U4.6 (D3), U8.18 (D7)

Commit message: [control] work in progress
Parts:
- removed U1, U2, U3, U4: 74LS163, symbol frits:74LS163
- removed U5, U6: 74LS244, symbol 74xx:74LS244
- added U1, U2: 74LS374, symbol 74xx:74LS374
Connections:
- net +5V: now also U1.20 (VCC), U2.20 (VCC)
- net GND: now also U1.10 (GND), U2.10 (GND)
- net ~{aregtoa}: now reaches U7.1 (OE)
- net ~{aregtoa}: now also U8.1 (OE)
- net ~{aregload}: now reaches U7.11 (Cp)
- net ~{aregload}: now also U8.11 (Cp)
- new net D0: U1.3 (D0)
- new net D1: U1.4 (D1)
- new net D10: U2.7 (D2)
- new net D11: U2.8 (D3)
- new net D12: U2.13 (D4)
- new net D13: U2.14 (D5)
- new net D14: U2.17 (D6)
- new net D15: U2.18 (D7)
- new net D2: U1.7 (D2)
- new net D3: U1.8 (D3)
- new net D4: U1.13 (D4)
- new net D5: U1.14 (D5)
- new net D6: U1.17 (D6)
- new net D7: U1.18 (D7)
- new net D8: U2.3 (D0)
- new net D9: U2.4 (D1)
- no-connect marks 1 -> 0
Other:
- moved on the sheet: U7, U8
